File: hardware/uPTP.kicad_pcb (KiCad board)
At the start: 4 copper layers, 40 x 50 mm, 79 parts, among them J1 PPS_UFL, J2 PPS_SMA, J3 LED, J4 UART_HDR, J5 HC-RJ45-055-7, J6 AUX_PWR, J7 PROG, U1 XC6206P332MR-G, U2 SI3404-A-GMR, U3 CH32V307WCU6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

Commit message: Correct misunderstandings, mostly there
Parts:
- moved R5 7.83 mm to (165.2, 83.5), turned to 0 degrees
- moved C13 7.63 mm to (150.5, 93.8)
- moved C14 7.63 mm to (153.0, 93.8)
- moved R14 7.51 mm to (148.8, 94.8)
- moved R15 7.50 mm to (148.8, 92.8)
- moved D7 7.22 mm to (158.2, 84.5), turned to 180 degrees
- moved C15 6.41 mm to (147.2, 93.0)
- moved D2 6.32 mm to (145.5, 93.0)
- moved R10 5.61 mm to (162.8, 91.5)
- moved L1 5.26 mm to (149.8, 87.8)
- moved C9 3.64 mm to (161.0, 91.0)
- moved C1 3.40 mm to (141.2, 82.0)
- moved C2 3.40 mm to (141.8, 83.5)
- moved C3 3.40 mm to (137.8, 86.0)
- moved D3 3.40 mm to (140.2, 89.0)
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Connections:
- C8 pad 2: /Ethernet and POE/ETH_ISENSE -> /Ethernet and POE/POE_VSS
- C9 pad 2: /Ethernet and POE/ETH_ISENSE -> /Ethernet and POE/POE_VSS
- H1 pad 1: GND -> unconnected-(H1-Pad1)
- H2 pad 1: GND -> unconnected-(H2-Pad1)
- J6 pad 1: /Ethernet and POE/ETH_POE_FILT_N -> /Ethernet and POE/ETH_ISENSE
- R10 pad 1: /Ethernet and POE/ETH_ISENSE -> /Ethernet and POE/POE_VSS
- R10 pad 2: /Ethernet and POE/POE_VSS -> /Ethernet and POE/ETH_ISENSE
- U2 pad 11: unconnected-(U2-NC-Pad11) -> /Ethernet and POE/ETH_POE_FILT_N
- U2 pad 12: unconnected-(U2-NC-Pad12) -> /Ethernet and POE/ETH_POE_FILT_N
- U2 pad 15: unconnected-(U2-NC-Pad15) -> /Ethernet and POE/ETH_POE_FILT_N
- U2 pad 17: unconnected-(U2-NC-Pad17) -> /Ethernet and POE/ETH_POE_FILT_N
- U2 pad 20: unconnected-(U2-NC-Pad20) -> /Ethernet and POE/ETH_POE_FILT_N
- U2 pad 7: unconnected-(U2-NC-Pad7) -> /Ethernet and POE/ETH_POE_FILT_N
Routing:
- net /Ethernet and POE/ETH_POE_FILT_P: track 0.00 -> 33.7 mm
- net /Ethernet and POE/ETH_ISENSE: track 0.00 -> 25.8 mm, vias 0 -> 2
- net /Ethernet and POE/ETH_5V_FB: track 0.00 -> 18.9 mm, vias 0 -> 2
- net /Ethernet and POE/ETH_POE_FILT_N: track 0.00 -> 12.3 mm, vias 0 -> 12
- net /Ethernet and POE/ETH_BUCK_SW: track 0.00 -> 10.6 mm
- net /Ethernet and POE/POE_VSS: track 0.00 -> 10.4 mm
- net /Ethernet and POE/ETH_POE_DET: track 0.00 -> 9.74 mm
- net GND: track 15.0 -> 20.8 mm
- net /Ethernet and POE/ETH_AUX: track 0.00 -> 5.81 mm
- net /Ethernet and POE/RFREQ: track 0.00 -> 3.01 mm
- net /Ethernet and POE/ETH_EROUT: track 0.00 -> 2.34 mm
- net /Ethernet and POE/ETH_VDD: track 0.00 -> 1.88 mm
- net /Ethernet and POE/ETH_C_MID: track 0.00 -> 1.82 mm
- net /Ethernet and POE/ETH_POE_CLASS: track 0.00 -> 1.33 mm
- net /Ethernet and POE/ETH_EROUT_RC: track 0.00 -> 0.97 mm
- added copper zone on F.Cu, net /Ethernet and POE/ETH_POE_FILT_N
- added copper zone on In1.Cu, net /Ethernet and POE/ETH_POE_FILT_N

Commit message: Routed board, first draft
Parts:
- TP1: moved to F.Cu
- moved D3 3.91 mm to (142.8, 92.0)
- moved C3 3.75 mm to (140.0, 89.0)
- moved C1 3.61 mm to (143.2, 85.0)
- moved U1 3.61 mm to (142.8, 89.0)
- moved C2 3.47 mm to (143.5, 86.5)
- moved TP1 2.51 mm to (144.0, 82.5)
- moved JP1 0.25 mm to (151.8, 82.2), turned to 180 degrees
- moved C12 0.20 mm to (164.8, 92.7)
- moved R13 0.20 mm to (165.8, 92.7)
Routing:
- net +5V: track 9.57 -> 53.6 mm, vias 0 -> 3
- net /MCU/NMEA_UART_TX: track 0.00 -> 25.7 mm, vias 0 -> 1
- net /MCU/NMEA_UART_RX: track 0.00 -> 24.2 mm, vias 0 -> 1
- net /Ethernet and POE/ETH_POE_FILT_P: track 33.7 -> 44.1 mm, vias 0 -> 2
- net +3V3: track 19.0 -> 27.5 mm, vias 8 -> 12
- net GND: track 20.8 -> 25.5 mm, vias 7 -> 52
- net /Ethernet and POE/POE_VSS: track 10.4 -> 14.9 mm, vias 0 -> 2
- net /Ethernet and POE/ETH_POE_FILT_N: vias 12 -> 11
- added copper zone on B.Cu, net /Ethernet and POE/ETH_POE_FILT_N
- added copper zone on B.Cu, net GND
- added copper zone on F.Cu, net GND
