File: hardware/ethernet.kicad_sch (KiCad schematic)
At the start: 39 parts, among them J5 HC-RJ45-055-7, J6 AUX_PWR, U2 SI3404-A-GMR

Commit message: Fix BOM entries, should be good to go
Parts:
- C10, C6, C7: LCSC Part (none) -> C1525
- C12: LCSC Part (none) -> C1523
- R1, R2, R3, R4, R6: LCSC Part (none) -> C25133
- R10: LCSC Part (none) -> C2998063
- R13, R5: value 24.3k -> 24k; LCSC Part (none) -> C25769
- R14: value 11k -> 4.3k; LCSC Part (none) -> C25899
- R15: value 3.9k -> 12k; LCSC Part (none) -> C25752
- R7: LCSC Part (none) -> C170366
- TR1: value ~ -> Ethernet Magnetics
Changed lines of the file:
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@@
+			)
+		)
+		(property "LCSC Part" "C25133"
+			(at 69.85 154.94 0)
+			(effects
+				(font
+					(size 1.27 1.27)
+				)
+				(hide yes)
 			)
 		)
@@
 			)
 		)
+		(property "LCSC Part" "C25133"
+			(at 76.2 154.94 0)
+			(effects
+				(font
+					(size 1.27 1.27)
+				)
+				(hide yes)
+			)
+		)
 		(pin "1"
 		)
@@
 		)
 		(property "Description" "Resistor"
+			(at 88.9 154.94 0)
+			(effects
+				(font
+					(size 1.27 1.27)
+				)
+				(hide yes)
+			)
+		)
+		(property "LCSC Part" "C25133"
 			(at 88.9 154.94 0)
 			(effects
@@
 			)
 		)
+		(property "LCSC Part" "C25133"
+			(at 82.55 154.94 0)
+			(effects
+				(font
+					(size 1.27 1.27)
+				)
+				(hide yes)
+			)
+		)
 		(pin "1"
 		)
@@
 			)
 		)
-		(property "Value" "24.3k"
+		(property "Value" "24k"
 			(at 204.47 82.55 0)
 			(effects
@@
 			)
 		)
+		(property "LCSC Part" "C25769"
+			(at 203.2 81.28 0)
+			(effects
+				(font
+					(size 1.27 1.27)
+				)
+				(hide yes)
+			)
+		)
 		(pin "1"
 		)
@@
 			)
 		)
-		(property "Value" "11k"
+		(property "Value" "4.3k"
 			(at 242.57 52.07 0)
 			(effects
@@
 		)
 		(property "Description" "Resistor"
+			(at 241.3 50.8 0)
+			(effects
+				(font
+					(size 1.27 1.27)
+				)
+				(hide yes)
+			)
+		)
+		(property "LCSC Part" "C25899"
 			(at 241.3 50.8 0)
 			(effects
@@
 			)
 		)
+		(property "LCSC Part" "C1523"
+			(at 193.04 71.12 0)
+			(effects
+				(font
+					(size 1.27 1.27)
+				)
+				(hide yes)
+			)
+		)
 		(pin "1"
 		)
@@
 		)
 		(property "Description" "Unpolarized capacitor"
+			(at 182.88 81.28 0)
+			(effects
+				(font
+					(size 1.27 1.27)
+				)
+				(hide yes)
+			)
+		)
+		(property "LCSC Part" "C1525"
 			(at 182.88 81.28 0)
 			(effects
@@
 			)
 		)
+		(property "LCSC Part" "C25133"
+			(at 127 78.74 0)
+			(effects
+				(font
+					(size 1.27 1.27)
+				)
+				(hide yes)
+			)
+		)
 		(pin "1"
 		)
@@
 			)
 		)
+		(property "LCSC Part" "C1525"
+			(at 124.46 156.21 0)
+			(effects
+				(font
+					(size 1.27 1.27)
+				)
+				(hide yes)
+			)
+		)
 		(pin "1"
 		)
@@
 			)
 		)
+		(property "LCSC Part" "C2998063"
+			(at 170.18 49.53 0)
+			(effects
+				(font
+					(size 1.27 1.27)
+				)
+				(hide yes)
+			)
+		)
 		(pin "1"
 		)
@@
 			)
 		)
+		(property "LCSC Part" "C170366"
+			(at 153.67 44.45 0)
+			(effects
+				(font
+					(size 1.27 1.27)
+				)
+				(hide yes)
+			)
+		)
 		(pin "1"
 		)
@@
 			)
 		)
+		(property "LCSC Part" "C1525"
+			(at 116.84 156.21 0)
+			(effects
+				(font
+					(size 1.27 1.27)
+				)
+				(hide yes)
+			)
+		)
 		(pin "1"
 		)
@@
 			)
 		)
-		(property "Value" "~"
+		(property "Value" "Ethernet Magnetics"
 			(at 104.14 148.59 0)
 			(effects
@@
 					(size 1.27 1.27)
 				)
+				(hide yes)
 			)
 		)
@@
 			)
 		)
-		(property "Value" "3.9k"
+		(property "Value" "12k"
 			(at 242.57 77.47 0)
 			(effects
@@
 			)
 		)
+		(property "LCSC Part" "C25752"
+			(at 241.3 76.2 0)
+			(effects
+				(font
+					(size 1.27 1.27)
+				)
+				(hide yes)
+			)
+		)
 		(pin "1"
 		)
@@
 			)
 		)
-		(property "Value" "24.3k"
+		(property "Value" "24k"
 			(at 128.27 52.07 0)
 			(effects
@@
 			(at 127 50.8 0)
 			(effects
+				(font
+					(size 1.27 1.27)
+				)
+				(hide yes)
+			)
+		)
+		(property "LCSC Part" "C25769"
+			(at 127 50.8 0)
+			(effects

Commit message: First of listed hardware changes, need verification
Parts:
- removed R11, R12, R8, R9: 49.9, Resistor_SMD:R_0402_1005Metric, symbol Device:R
- added C26, C27, C28, C29: 10n, Capacitor_SMD:C_0402_1005Metric, symbol Device:C
Connections:
- net ETH_RX1: now also C29.1; no longer R4.1
- net ETH_RX2: now also C26.1; no longer R1.1
- net ETH_TX1: now also C28.1; no longer R3.1
- net ETH_TX2: now also C27.1; no longer R2.1
- new net: C26.2, R1.1
- new net: C27.2, R2.1
- new net: C29.2, R4.1
- new net: C28.2, R3.1
Other:
- note removed: "TVS Protection Necessary? RECOMMENDED FOR POE DESIGNS"
- note removed: "Unsure if Phy has built-in termination, placeholders close to MCU"
- moved on the sheet: C4, R1, R2, R3, R4
